File: PCB-Eagle/HMS_Olfactometer_v2.2.brd (EAGLE design)
At the start: 279.4 x 137.2 mm, 51 parts, among them IC1 ULQ2803A, IC10 ULQ2803A3, IC3 ULQ2803A, IC4 ULQ2803A, IC5 ULQ2803A, IC6 ULQ2803A, IC8 ULQ2803A

Commit message: [PCB] Small changes to layout and silkscreen; Version 2.2
Parts:
- moved 5V 8.03 mm to (22.1, 123.3)
- moved C4 7.62 mm to (27.9, 105.4)
- moved C5 7.62 mm to (20.3, 105.4)
- moved DC_5V 7.62 mm to (24.1, 110.5)
Routing:
- net +5V: track 70.9 -> 67.6 mm
- net +12V: track 1554.7 -> 1557.8 mm
Other:
- board text added: "P7805-500"
- board text added: "Teensy 3.5 or 4.1"
- board text added: "The Olfactory Delivery Board v2.2 October 2023, OM HMS Research Instrumentation Core"
- board text removed: "Teensy 3.5"
- board text removed: "The Olfactory Delivery Board v2.1 October 2018, OM HMS Research Instrumentation Core"

Commit message: [PCB] Update silkscreen; Add redundant GND trace to fix air wire
Routing:
- net GND: track 0.00 -> 41.1 mm, vias 2 -> 6
- net V35: track 163.9 -> 168.0 mm
- net +5V: track 67.6 -> 69.9 mm
Other:
- board text added: "Not needed if Teensy gets power from USB. If used, must cut trace on Teensy between V_IN and V_USB."
- board text added: "Teensy Power"
- board text removed: "(Cut trace between V_IN and V_USB.)"
Changed lines of the file:
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@@
 <text x="20.32" y="114.935" size="1.016" layer="25" ratio="10">VX7805-500</text>
 <text x="52.07" y="89.535" size="1.778" layer="21" ratio="15" rot="R90">Teensy 3.5 or 4.1</text>
-<text x="53.975" y="84.455" size="1.27" layer="21" ratio="10" rot="R90">(Cut trace between V_IN and V_USB.)</text>
+<text x="35.56" y="125.73" size="1.016" layer="21" ratio="10" rot="SR270">Not needed if Teensy gets power from USB.
+If used, must cut trace on Teensy
+between V_IN and V_USB.</text>
 <text x="14.605" y="132.08" size="1.778" layer="21" rot="SR270">BNC 1</text>
 <text x="14.605" y="105.41" size="1.778" layer="21" rot="SR270">BNC 2</text>
 <text x="20.32" y="113.665" size="1.016" layer="25" ratio="10">P7805-500</text>
+<wire x1="17.145" y1="129.54" x2="43.18" y2="129.54" width="0.1524" layer="25" style="shortdash"/>
+<wire x1="43.18" y1="129.54" x2="43.18" y2="93.98" width="0.1524" layer="25" style="shortdash"/>
+<wire x1="43.18" y1="93.98" x2="17.145" y2="93.98" width="0.1524" layer="25" style="shortdash"/>
+<wire x1="17.145" y1="93.98" x2="17.145" y2="129.54" width="0.1524" layer="25" style="shortdash"/>
+<text x="40.64" y="125.73" size="1.778" layer="25" rot="SR270">Teensy Power</text>
 </plain>
 <attributes>
@@
 <contactref element="IC10" pad="5"/>
 <contactref element="IC10" pad="6"/>
+<wire x1="63.5" y1="92.71" x2="53.34" y2="92.71" width="0.2032" layer="1"/>
+<via x="53.34" y="92.71" extent="1-16" drill="0.3556"/>
+<wire x1="53.34" y1="92.71" x2="53.34" y2="96.52" width="0.2032" layer="16"/>
+<via x="53.34" y="96.52" extent="1-16" drill="0.3556"/>
+<wire x1="53.34" y1="96.52" x2="45.085" y2="96.52" width="0.2032" layer="1"/>
+<via x="45.085" y="96.52" extent="1-16" drill="0.3556"/>
+<wire x1="45.085" y1="96.52" x2="34.29" y2="85.725" width="0.2032" layer="16"/>
+<wire x1="34.29" y1="85.725" x2="34.29" y2="85.09" width="0.2032" layer="16"/>
+<via x="34.29" y="85.09" extent="1-16" drill="0.3556"/>
+<wire x1="34.29" y1="85.09" x2="33.15" y2="83.95" width="0.2032" layer="1"/>
+<wire x1="33.15" y1="83.95" x2="31.75" y2="83.95" width="0.2032" layer="1"/>
 <wire x1="87.63" y1="107.95" x2="63.5" y2="92.71" width="0" layer="19" extent="1-1"/>
 </signal>
@@
 <contactref element="DC_5V" pad="3"/>
 <contactref element="C4" pad="1"/>
-<wire x1="63.5" y1="128.27" x2="46.99" y2="128.27" width="0.6096" layer="1"/>
-<wire x1="46.99" y1="128.27" x2="31.75" y2="113.03" width="0.6096" layer="1"/>
-<wire x1="31.75" y1="113.03" x2="31.75" y2="109.22" width="0.6096" layer="1"/>
+<wire x1="63.5" y1="128.27" x2="61.595" y2="130.175" width="0.6096" layer="1"/>
+<wire x1="61.595" y1="130.175" x2="47.625" y2="130.175" width="0.6096" layer="1"/>
+<wire x1="47.625" y1="130.175" x2="31.75" y2="114.3" width="0.6096" layer="1"/>
+<wire x1="31.75" y1="114.3" x2="31.75" y2="109.22" width="0.6096" layer="1"/>
 <wire x1="29.34" y1="105.41" x2="29.34" y2="106.81" width="0.6096" layer="1"/>
 <wire x1="31.75" y1="109.22" x2="29.34" y2="106.81" width="0.6096" layer="1"/>
@@
 <wire x1="48.26" y1="101.3968" x2="50.8" y2="103.9368" width="0.2032" layer="1"/>
 <wire x1="47.8536" y1="101.3968" x2="48.26" y2="101.3968" width="0.2032" layer="1"/>
-<wire x1="47.1424" y1="100.6856" x2="47.8536" y2="101.3968" width="0.2032" layer="1"/>
-<wire x1="47.1424" y1="94.8944" x2="47.1424" y2="100.6856" width="0.2032" layer="1"/>
-<wire x1="48.1584" y1="93.8784" x2="47.1424" y2="94.8944" width="0.2032" layer="1"/>
-<wire x1="49.6824" y1="93.8784" x2="48.1584" y2="93.8784" width="0.2032" layer="1"/>
+<wire x1="43.9674" y1="97.5106" x2="47.8536" y2="101.3968" width="0.2032" layer="1"/>
+<wire x1="43.9674" y1="95.5294" x2="43.9674" y2="97.5106" width="0.2032" layer="1"/>
+<wire x1="45.6184" y1="93.8784" x2="43.9674" y2="95.5294" width="0.2032" layer="1"/>
+<wire x1="49.6824" y1="93.8784" x2="45.6184" y2="93.8784" width="0.2032" layer="1"/>
 <wire x1="55.88" y1="87.6808" x2="49.6824" y2="93.8784" width="0.2032" layer="1"/>
 <wire x1="184.0992" y1="123.1392" x2="184.15" y2="123.19" width="0.2032" layer="16"/>

Commit message: [PCB] Fix the actual ground-plane bug in v2.2
Routing:
- net GND: track 41.1 -> 51.9 mm, vias 6 -> 4
Changed lines of the file:
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@@
 <contactref element="IC10" pad="5"/>
 <contactref element="IC10" pad="6"/>
-<wire x1="63.5" y1="92.71" x2="53.34" y2="92.71" width="0.2032" layer="1"/>
-<via x="53.34" y="92.71" extent="1-16" drill="0.3556"/>
-<wire x1="53.34" y1="92.71" x2="53.34" y2="96.52" width="0.2032" layer="16"/>
-<via x="53.34" y="96.52" extent="1-16" drill="0.3556"/>
-<wire x1="53.34" y1="96.52" x2="45.085" y2="96.52" width="0.2032" layer="1"/>
-<via x="45.085" y="96.52" extent="1-16" drill="0.3556"/>
-<wire x1="45.085" y1="96.52" x2="34.29" y2="85.725" width="0.2032" layer="16"/>
-<wire x1="34.29" y1="85.725" x2="34.29" y2="85.09" width="0.2032" layer="16"/>
-<via x="34.29" y="85.09" extent="1-16" drill="0.3556"/>
-<wire x1="34.29" y1="85.09" x2="33.15" y2="83.95" width="0.2032" layer="1"/>
-<wire x1="33.15" y1="83.95" x2="31.75" y2="83.95" width="0.2032" layer="1"/>
-<wire x1="87.63" y1="107.95" x2="63.5" y2="92.71" width="0" layer="19" extent="1-1"/>
+<wire x1="87.63" y1="107.95" x2="90.17" y2="110.49" width="0.3048" layer="16"/>
+<wire x1="90.17" y1="110.49" x2="90.17" y2="125.73" width="0.3048" layer="16"/>
+<via x="90.17" y="125.73" extent="1-16" drill="0.3556"/>
+<wire x1="90.17" y1="125.73" x2="90.17" y2="129.54" width="0.3048" layer="1"/>
+<wire x1="90.17" y1="129.54" x2="88.9" y2="130.81" width="0.3048" layer="1"/>
+<wire x1="68.58466875" y1="130.81" x2="66.04466875" y2="128.27" width="0.3048" layer="1"/>
+<via x="66.04466875" y="128.27" extent="1-16" drill="0.3556"/>
+<wire x1="66.04466875" y1="128.27" x2="63.50466875" y2="125.73" width="0.3048" layer="16"/>
+<wire x1="63.50466875" y1="125.73" x2="63.5" y2="125.73" width="0.3048" layer="16"/>
+<wire x1="88.9" y1="130.81" x2="68.58466875" y2="130.81" width="0.3048" layer="1"/>
 </signal>
 <signal name="+12V" class="1">
