File: PCB-KiCAD/HMS Olfactometer.kicad_pcb (KiCad board)
At the start: 2 copper layers, 1 part

Commit message: [PCB] More work on PCB v3
Parts:
- added H1: MountingHole, MountingHole:MountingHole_3.2mm_M3, F.Cu at (155.6, 164.5)
- added H10: MountingHole, MountingHole:MountingHole_3.2mm_M3, F.Cu at (225.4, 128.9)
- added H11: MountingHole, MountingHole:MountingHole_3.2mm_M3, F.Cu at (337.1, 128.9)
- added H12: MountingHole, MountingHole:MountingHole_3.2mm_M3, F.Cu at (225.4, 95.9)
- added H2: MountingHole, MountingHole:MountingHole_3.2mm_M3, F.Cu at (267.3, 164.5)
- added H3: MountingHole, MountingHole:MountingHole_3.2mm_M3, F.Cu at (267.3, 95.9)
- added H4: MountingHole, MountingHole:MountingHole_3.2mm_M3, F.Cu at (155.6, 128.9)
- added H5: MountingHole, MountingHole:MountingHole_3.2mm_M3, F.Cu at (267.3, 128.9)
- added H6: MountingHole, MountingHole:MountingHole_3.2mm_M3, F.Cu at (155.6, 95.9)
- added H7: MountingHole, MountingHole:MountingHole_3.2mm_M3, F.Cu at (225.4, 164.5)
- added H8: MountingHole, MountingHole:MountingHole_3.2mm_M3, F.Cu at (337.1, 164.5)
- added H9: MountingHole, MountingHole:MountingHole_3.2mm_M3, F.Cu at (337.1, 95.9)
- added J1: Conn_01x24, Connector_PinHeader_2.54mm:PinHeader_1x24_P2.54mm_Vertical, F.Cu at (162.6, 142.2)
- added J10: Conn_01x02, Connector_PinHeader_2.54mm:PinHeader_1x02_P2.54mm_Vertical, F.Cu at (316.6, 45.7)
- added J11: Conn_01x02, Connector_PinHeader_2.54mm:PinHeader_1x02_P2.54mm_Vertical, F.Cu at (271.8, 58.4)
- added J12: Conn_01x02, Connector_PinHeader_2.54mm:PinHeader_1x02_P2.54mm_Vertical, F.Cu at (286.1, 58.4)
- added J13: Conn_01x02, Connector_PinHeader_2.54mm:PinHeader_1x02_P2.54mm_Vertical, F.Cu at (301.3, 58.4)
- added J14: Conn_01x02, Connector_PinHeader_2.54mm:PinHeader_1x02_P2.54mm_Vertical, F.Cu at (316.6, 58.4)
- added J15: 24 V DC, Connector_BarrelJack:BarrelJack_CUI_PJ-102AH_Horizontal, F.Cu at (76.2, 101.6)
- added J16: Conn_01x06, Connector_Molex:Molex_CLIK-Mate_502382-0670_1x06-1MP_P1.25mm_Vertical, F.Cu at (78.7, 144.8)
- added J17: Conn_01x06, Connector_Molex:Molex_CLIK-Mate_502382-0670_1x06-1MP_P1.25mm_Vertical, F.Cu at (78.7, 160.0)
- added J18: Conn_01x06, Connector_Molex:Molex_CLIK-Mate_502382-0670_1x06-1MP_P1.25mm_Vertical, F.Cu at (104.1, 144.8)
- added J19: Conn_01x06, Connector_Molex:Molex_CLIK-Mate_502382-0670_1x06-1MP_P1.25mm_Vertical, F.Cu at (104.1, 160.0)
- added J2: Conn_01x24, Connector_PinHeader_2.54mm:PinHeader_1x24_P2.54mm_Vertical, F.Cu at (274.2, 142.2)
- added J20: Conn_Coaxial, Connector_Coaxial:BNC_Amphenol_B6252HB-NPP3G-50_Horizontal, F.Cu at (134.6, 50.8)
- added J21: Conn_Coaxial, Connector_Coaxial:BNC_Amphenol_B6252HB-NPP3G-50_Horizontal, F.Cu at (162.6, 50.8)
- added J22: Conn_Coaxial, Connector_Coaxial:BNC_Amphenol_B6252HB-NPP3G-50_Horizontal, F.Cu at (190.5, 50.8)
- added J23: Conn_Coaxial, Connector_Coaxial:BNC_Amphenol_B6252HB-NPP3G-50_Horizontal, F.Cu at (218.4, 50.8)
- added J24: Conn_01x16, Connector_PinHeader_2.54mm:PinHeader_1x16_P2.54mm_Vertical, F.Cu at (83.8, 40.6)
- added J25: I2C_STANDARDQWIIC, SparkFun-Connectors:1X04_1MM_RA, F.Cu at (74.8, 61.2)
- added J3: Conn_01x24, Connector_PinHeader_2.54mm:PinHeader_1x24_P2.54mm_Vertical, F.Cu at (274.2, 73.7)
- added J4: Conn_01x24, Connector_PinHeader_2.54mm:PinHeader_1x24_P2.54mm_Vertical, F.Cu at (162.6, 106.7)
- added J5: Conn_01x24, Connector_PinHeader_2.54mm:PinHeader_1x24_P2.54mm_Vertical, F.Cu at (274.2, 106.7)
- added J6: Conn_01x24, Connector_PinHeader_2.54mm:PinHeader_1x24_P2.54mm_Vertical, F.Cu at (162.6, 73.7)
- added J7: Conn_01x02, Connector_PinHeader_2.54mm:PinHeader_1x02_P2.54mm_Vertical, F.Cu at (271.8, 45.7)
- added J8: Conn_01x02, Connector_PinHeader_2.54mm:PinHeader_1x02_P2.54mm_Vertical, F.Cu at (286.1, 45.7)
- added J9: Conn_01x02, Connector_PinHeader_2.54mm:PinHeader_1x02_P2.54mm_Vertical, F.Cu at (301.3, 45.7)
- added JP1: SolderJumper_2_Open, Jumper:SolderJumper-2_P1.3mm_Open_RoundedPad1.0x1.5mm, F.Cu at (86.4, 118.7)
- added R1: R, Resistor_THT:R_Axial_DIN0207_L6.3mm_D2.5mm_P10.16mm_Horizontal, F.Cu at (97.1, 132.1)
- added R2: R, Resistor_THT:R_Axial_DIN0207_L6.3mm_D2.5mm_P10.16mm_Horizontal, F.Cu at (101.1, 132.1)
- added R3: R, Resistor_THT:R_Axial_DIN0207_L6.3mm_D2.5mm_P10.16mm_Horizontal, F.Cu at (105.2, 132.1)
- added R4: R, Resistor_THT:R_Axial_DIN0207_L6.3mm_D2.5mm_P10.16mm_Horizontal, F.Cu at (109.2, 132.1)
- added SW1: SW_SPST, Button_Switch_THT:SW_SPST_Omron_B3F-315x_Angled, F.Cu at (71.7, 119.4)
- added U1: Teensy4.0, teensy:Teensy40_noInternalPins, F.Cu at (104.1, 59.7)
- added U10: ULN2803A, Package_DIP:DIP-18_W7.62mm, F.Cu at (252.0, 106.7)
- added U11: MCP23008-xP, Package_DIP:DIP-18_W7.62mm, F.Cu at (238.7, 106.7)
- added U12: ULN2803A, Package_DIP:DIP-18_W7.62mm, F.Cu at (140.3, 73.7)
- added U13: MCP23008-xP, Package_DIP:DIP-18_W7.62mm, F.Cu at (127.0, 73.7)
- added U14: ULN2803A, Package_DIP:DIP-18_W7.62mm, F.Cu at (251.5, 40.6)
- added U15: MCP23008-xP, Package_DIP:DIP-18_W7.62mm, F.Cu at (238.8, 40.6)
- added U16: R-78B12-2.0, Converter_DCDC:Converter_DCDC_RECOM_R-78B-2.0_THT, F.Cu at (99.1, 99.1)
- added U2: ULN2803A, Package_DIP:DIP-18_W7.62mm, F.Cu at (140.3, 142.2)
- added U3: MCP23008-xP, Package_DIP:DIP-18_W7.62mm, F.Cu at (127.0, 142.2)
- added U4: ULN2803A, Package_DIP:DIP-18_W7.62mm, F.Cu at (252.0, 142.2)
- added U5: MCP23008-xP, Package_DIP:DIP-18_W7.62mm, F.Cu at (238.7, 142.2)
- added U6: ULN2803A, Package_DIP:DIP-18_W7.62mm, F.Cu at (252.0, 73.7)
- added U7: MCP23008-xP, Package_DIP:DIP-18_W7.62mm, F.Cu at (238.7, 73.7)
- added U8: ULN2803A, Package_DIP:DIP-18_W7.62mm, F.Cu at (140.3, 106.7)
- added U9: MCP23008-xP, Package_DIP:DIP-18_W7.62mm, F.Cu at (127.0, 106.7)
- moved G1 74.6 mm to (172.4, 177.8)
Routing:
- net +12V: track 0.00 -> 685.7 mm
- net Net-(J3-Pin_22): track 0.00 -> 75.3 mm
- net Net-(J2-Pin_22): track 0.00 -> 75.3 mm
- net Net-(J6-Pin_22): track 0.00 -> 75.3 mm
- net Net-(J5-Pin_22): track 0.00 -> 75.3 mm
- net Net-(J4-Pin_22): track 0.00 -> 75.3 mm
- net Net-(J1-Pin_22): track 0.00 -> 75.3 mm
- net Net-(J6-Pin_19): track 0.00 -> 66.6 mm
- net Net-(J5-Pin_19): track 0.00 -> 66.6 mm
- net Net-(J4-Pin_19): track 0.00 -> 66.6 mm
- net Net-(J3-Pin_19): track 0.00 -> 66.6 mm
- net Net-(J2-Pin_19): track 0.00 -> 66.6 mm
- net Net-(J1-Pin_19): track 0.00 -> 66.6 mm
- net Net-(J6-Pin_16): track 0.00 -> 58.0 mm
- net Net-(J3-Pin_16): track 0.00 -> 58.0 mm
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Other:
- board outline added: 279.4 x 137.2 mm
- board text added: "1"
- board text added: "12V DC-DC Converter"
- board text added: "16"
- board text added: "17"
- board text added: "2"
- board text added: "24"
- board text added: "25"
- board text added: "3"
- board text added: "32"
- board text added: "33"
- board text added: "4"
- board text added: "40"
- board text added: "41"
- board text added: "48"
- board text added: "5"
- board text added: "6"
- board text added: "7"
- board text added: "8"
- board text added: "9"
- board text added: "Aux 1"
- board text added: "HMS Olfactometer Driver"
- board text added: "HMS Research Instrumentation Core v4.0 - OM - Dec. 2024"
- board text added: "I2C"
- board text added: "On/Off Switch"
- board text added: "Sensirion MFCs"
- board text added: "Teensy 4.0 or 3.2"
- board text removed: "HMS Research Instrumentation Core v1.0 - Date"
- board text removed: "Name of PCB"

Commit message: Finalize PCB v3; Renumber to v4
Parts:
- added C1: C, Capacitor_THT:CP_Radial_Tantal_D6.0mm_P2.50mm, F.Cu at (52.1, 83.8)
- added C2: C, Capacitor_THT:CP_Radial_Tantal_D6.0mm_P2.50mm, F.Cu at (74.9, 83.8)
- added D1: LED, LED_THT:LED_D3.0mm, F.Cu at (62.2, 100.3)
- added H13: MountingHole, MountingHole:MountingHole_3.2mm_M3, F.Cu at (38.1, 38.1)
- added H14: MountingHole, MountingHole:MountingHole_3.2mm_M3, F.Cu at (38.1, 165.1)
- added H15: MountingHole, MountingHole:MountingHole_3.2mm_M3, F.Cu at (304.8, 38.1)
- added H16: MountingHole, MountingHole:MountingHole_3.2mm_M3, F.Cu at (304.8, 139.7)
- added H17: MountingHole, MountingHole:MountingHole_3.2mm_M3, F.Cu at (196.8, 165.1)
- added H18: MountingHole, MountingHole:MountingHole_3.2mm_M3, F.Cu at (196.8, 38.1)
- added R16: 10k, Resistor_THT:R_Axial_DIN0207_L6.3mm_D2.5mm_P10.16mm_Horizontal, F.Cu at (110.5, 61.0)
- added R5: 10k, Resistor_THT:R_Axial_DIN0207_L6.3mm_D2.5mm_P10.16mm_Horizontal, F.Cu at (42.4, 44.5)
- added R6: 10k, Resistor_THT:R_Axial_DIN0207_L6.3mm_D2.5mm_P10.16mm_Horizontal, F.Cu at (42.4, 72.4)
- added R7: 10k, Resistor_THT:R_Axial_DIN0207_L6.3mm_D2.5mm_P10.16mm_Horizontal, F.Cu at (85.1, 85.1)
- added R8: 10k, Resistor_THT:R_Axial_DIN0207_L6.3mm_D2.5mm_P10.16mm_Horizontal, F.Cu at (105.4, 61.0)
- added TP1: 24V, TestPoint:TestPoint_Loop_D1.80mm_Drill1.0mm_Beaded, F.Cu at (45.7, 88.9)
- added TP2: 12V, TestPoint:TestPoint_Loop_D1.80mm_Drill1.0mm_Beaded, F.Cu at (68.6, 101.6)
- added TP3: Gnd, TestPoint:TestPoint_Loop_D1.80mm_Drill1.0mm_Beaded, F.Cu at (81.3, 162.6)
- added TP4: 3V3, TestPoint:TestPoint_Loop_D1.80mm_Drill1.0mm_Beaded, F.Cu at (83.8, 40.6)
- J15: value 24 V DC -> +24 VDC
- J16: value Conn_01x06 -> MFC 1; footprint Connector_Molex:Molex_CLIK-Mate_502382-0670_1x06-1MP_P1.25mm_Vertical -> Connector_Sensirion:CONN_50556806xx_MOL
- J17: value Conn_01x06 -> MFC 3; footprint Connector_Molex:Molex_CLIK-Mate_502382-0670_1x06-1MP_P1.25mm_Vertical -> Connector_Sensirion:CONN_50556806xx_MOL
- J18: value Conn_01x06 -> MFC 2; footprint Connector_Molex:Molex_CLIK-Mate_502382-0670_1x06-1MP_P1.25mm_Vertical -> Connector_Sensirion:CONN_50556806xx_MOL
- J19: value Conn_01x06 -> MFC 4; footprint Connector_Molex:Molex_CLIK-Mate_502382-0670_1x06-1MP_P1.25mm_Vertical -> Connector_Sensirion:CONN_50556806xx_MOL
- JP1: footprint Jumper:SolderJumper-2_P1.3mm_Open_RoundedPad1.0x1.5mm -> Jumper:SolderJumper-2_P1.3mm_Bridged_RoundedPad1.0x1.5mm
- R1: value R -> 560
- R2: value R -> 1.2k
- R3: value R -> 2.7k
- SW1: value SW_SPST -> 500SSP1S1M6QEA; footprint Button_Switch_THT:SW_SPST_Omron_B3F-315x_Angled -> OnOff_Switch:SW_500SSP1S1M6QEA
- U11, U13, U15, U3, U5, U7, U9: value MCP23008-xP -> MCP23008
- moved G1 123.0 mm to (81.3, 95.2), turned to -90 degrees
- moved R3 66.4 mm to (48.3, 166.4), turned to 0 degrees
- moved R2 61.0 mm to (48.3, 162.6), turned to 0 degrees
- moved R1 55.6 mm to (48.3, 158.8), turned to 0 degrees
- moved R4 54.0 mm to (62.2, 105.4), turned to -90 degrees
- moved U16 41.4 mm to (61.0, 82.9)
- moved J15 40.3 mm to (40.6, 82.5)
- moved J19 39.7 mm to (65.5, 150.9)
- moved J18 39.7 mm to (65.5, 135.6)
- moved JP1 39.4 mm to (48.3, 108.6)
- moved J17 37.8 mm to (42.0, 150.9)
- moved J16 37.8 mm to (42.0, 135.6)
- moved SW1 37.1 mm to (37.3, 105.4), turned to 90 degrees
- moved J2 35.9 mm to (238.7, 137.2)
- moved H2 35.9 mm to (231.7, 159.4)
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Connections:
- J16 pad 5: Net-(J16-Pin_5) -> GND
- J24 pad 15: Net-(J24-Pin_15) -> +3.3V
- R1 pad 1: Net-(J16-Pin_5) -> Net-(J18-Pin_5)
- R3 pad 1: Net-(J18-Pin_5) -> Net-(J19-Pin_5)
- R4 pad 1: Net-(J19-Pin_5) -> Net-(D1-K)
- U1 pad 14: Net-(J24-Pin_15) -> unconnected-(U1-12_MISO_MQSL-Pad14)
- U11 pad 6: unconnected-(U11-~{RESET}-Pad6) -> RESET
- U13 pad 3: +3.3V -> GND
- U13 pad 5: +3.3V -> GND
- U13 pad 6: unconnected-(U13-~{RESET}-Pad6) -> RESET
- U14 pad 10: +3.3V -> +12V
- U15 pad 6: unconnected-(U15-~{RESET}-Pad6) -> RESET
- U3 pad 4: GND -> +3.3V
- U3 pad 6: unconnected-(U3-~{RESET}-Pad6) -> RESET
- U5 pad 3: GND -> +3.3V
- U5 pad 6: unconnected-(U5-~{RESET}-Pad6) -> RESET
- U7 pad 5: GND -> +3.3V
- U7 pad 6: unconnected-(U7-~{RESET}-Pad6) -> RESET
- U9 pad 4: +3.3V -> GND
- U9 pad 6: unconnected-(U9-~{RESET}-Pad6) -> RESET
Routing:
- net +3.3V: track 0.00 -> 714.6 mm
- net +12V: track 685.7 -> 1171.8 mm
- net RESET: track 0.00 -> 377.3 mm
- net SCL-0: track 0.00 -> 339.6 mm
- net SDA-0: track 0.00 -> 339.0 mm, vias 0 -> 1
- net /SDA-1: track 0.00 -> 177.7 mm, vias 0 -> 3
- net /SCL-1: track 0.00 -> 174.3 mm, vias 0 -> 2
- net +24V: track 0.00 -> 141.8 mm
- net Net-(J23-In): track 0.00 -> 116.1 mm
- net Net-(J22-In): track 0.00 -> 87.2 mm
- net Net-(J14-Pin_1): track 0.00 -> 73.4 mm
- net Net-(J10-Pin_1): track 0.00 -> 72.4 mm
- net Net-(J13-Pin_1): track 0.00 -> 55.6 mm
- net Net-(J9-Pin_1): track 0.00 -> 54.6 mm
- net Net-(J21-In): track 0.00 -> 52.9 mm
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- added copper zone on B.Cu, net GND
- added copper zone on F.Cu, net GND
Other:
- board text added: "3V3"
- board text added: "Aux Valves"
- board text added: "BNC-1"
- board text added: "BNC-2"
- board text added: "BNC-3"
- board text added: "BNC-4"
- board text added: "Gnd"
- board text added: "MFCs, Qwiic"
- board text added: "OFF"
- board text added: "ON"
- board text added: "On/Off Switch is optional. Cut solder jumper if using switch."
- board text added: "P0"
- board text added: "P1"
- board text added: "P10"
- board text added: "P11"
- board text added: "P2"
- board text added: "P3"
- board text added: "P4"
- board text added: "P5"
- board text added: "P6"
- board text added: "P7"
- board text added: "P8"
- board text added: "P9"
- board text added: "SCL-0"
- board text added: "SCL-1"
- board text added: "SDA-0"
- board text added: "SDA-1"
- board text added: "Valve Manifolds"
- board text added: "Valves"
- board text removed: "Aux 1"
- board text removed: "On/Off Switch"
