File: PCB-KiCAD/Valve_Module_8x_I2C.kicad_sch (KiCad schematic)
At the start: 3 parts, among them J1 Conn_01x24, U2 ULN2803A, U3 MCP23008-xP

Commit message: [PCB] More work on PCB v3
Parts:
- added H1, H7: MountingHole, MountingHole:MountingHole_3.2mm_M3, symbol Mechanical:MountingHole
- J1: footprint (none) -> Connector_PinHeader_2.54mm:PinHeader_1x24_P2.54mm_Vertical
- U2: footprint (none) -> Package_DIP:DIP-18_W7.62mm
Connections:
- net +3.3V: no longer J1.11 (Pin_11), J1.14 (Pin_14), J1.17 (Pin_17), J1.2 (Pin_2), J1.20 (Pin_20), J1.23 (Pin_23), J1.5 (Pin_5), J1.8 (Pin_8), U2.10 (COM)
- net at U2.1 (I1): now also U3.17 (GP7); no longer U3.10 (GP0)
- net at U2.2 (I2): now also U3.16 (GP6); no longer U3.11 (GP1)
- net at U2.3 (I3): now also U3.15 (GP5); no longer U3.12 (GP2)
- net at U2.4 (I4): now also U3.14 (GP4); no longer U3.13 (GP3)
- net at U2.5 (I5): now also U3.13 (GP3); no longer U3.14 (GP4)
- net at U2.6 (I6): now also U3.12 (GP2); no longer U3.15 (GP5)
- net at U2.7 (I7): now also U3.11 (GP1); no longer U3.16 (GP6)
- net at U2.8 (I8): now also U3.10 (GP0); no longer U3.17 (GP7)
- net A2: now reaches U3.3 (A2)
- net A1: now reaches U3.4 (A1)
- net A0: now reaches U3.5 (A0)
- new net +12V: J1.11 (Pin_11), J1.14 (Pin_14), J1.17 (Pin_17), J1.2 (Pin_2), J1.20 (Pin_20), J1.23 (Pin_23), J1.5 (Pin_5), J1.8 (Pin_8), U2.10 (COM)
- no-connect marks 8 -> 10
Other:
- moved on the sheet: U3

Commit message: Finalize PCB v3; Renumber to v4
Parts:
- U3: value MCP23008-xP -> MCP23008
Connections:
- net RESET: now reaches U3.6 (~{RESET})
- no-connect marks 10 -> 9
Changed lines of the file:
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@@
-	)
-	(no_connect
-		(at 35.56 35.56)
 	)
 	(no_connect
@@
 		(pts
 			(xy 91.44 60.96) (xy 91.44 58.42)
+		)
+		(stroke
+			(width 0)
+			(type default)
+		)
+	)
+	(wire
+		(pts
+			(xy 33.02 35.56) (xy 35.56 35.56)
 		)
 		(stroke
@@
 		(property "Intersheetrefs" "${INTERSHEET_REFS}"
 			(at 23.6848 40.64 0)
+			(effects
+				(font
+					(size 1.27 1.27)
+				)
+				(justify right)
+				(hide yes)
+			)
+		)
+	)
+	(global_label "RESET"
+		(shape input)
+		(at 33.02 35.56 180)
+		(fields_autoplaced yes)
+		(effects
+			(font
+				(size 1.27 1.27)
+			)
+			(justify right)
+		)
+		(property "Intersheetrefs" "${INTERSHEET_REFS}"
+			(at 24.2897 35.56 0)
 			(effects
 				(font
@@
 			)
 		)
-		(property "Value" "MCP23008-xP"
+		(property "Value" "MCP23008"
 			(at 50.4541 30.48 0)
 			(effects
