File: PCB-v4-KiCAD/Standalone_Valves_8x_I2C.kicad_sch (KiCad schematic)
At the start: 10 parts, among them J10 Conn_01x02, J11 Conn_01x02, J12 Conn_01x02, J13 Conn_01x02, J14 Conn_01x02, J7 Conn_01x02, J8 Conn_01x02, J9 Conn_01x02, U14 ULN2803A, U15 MCP23008

Commit message: [PCB] Fix pinout of Sensirion connector; Bump version to v4.1
Other:
- title: (none) -> HMS Multichannel Olfactometer Driver
Changed lines of the file:
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@@
 	(paper "USLetter")
 	(title_block
+		(title "HMS Multichannel Olfactometer Driver")
+		(date "2025-01-23")
+		(rev "4.1")
 		(company "HMS Research Instrumentation Core")
 	)
@@
 		(shape input)
 		(at 38.1 60.96 180)
-		(fields_autoplaced yes)
 		(effects
 			(font
@@
 		(shape input)
 		(at 38.1 58.42 180)
-		(fields_autoplaced yes)
 		(effects
 			(font
@@
 		(shape input)
 		(at 38.1 55.88 180)
-		(fields_autoplaced yes)
 		(effects
 			(font
