File: PCB-v4-KiCAD/Valve_Module_8x_I2C.kicad_sch (KiCad schematic)
At the start: 5 parts, among them J1 Conn_01x24, U2 ULN2803A, U3 MCP23008

Commit message: [PCB] Fix pinout of Sensirion connector; Bump version to v4.1
Other:
- title: (none) -> HMS Multichannel Olfactometer Driver
Changed lines of the file:
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@@
 	(paper "USLetter")
 	(title_block
+		(title "HMS Multichannel Olfactometer Driver")
+		(date "2025-01-23")
+		(rev "4.1")
 		(company "HMS Research Instrumentation Core")
 	)
@@
 		(shape input)
 		(at 33.02 55.88 180)
-		(fields_autoplaced yes)
 		(effects
 			(font
@@
 		(shape input)
 		(at 33.02 50.8 180)
-		(fields_autoplaced yes)
 		(effects
 			(font
@@
 		(shape input)
 		(at 33.02 53.34 180)
-		(fields_autoplaced yes)
 		(effects
 			(font

Commit message: Change silkscreen version number to 4.1; Update KiCad version
Parts:
- renumbered H7 to H12, H1 to H6, J1 to J6, U2 to U12, U3 to U13
Changed lines of the file:
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@@
 (kicad_sch
-	(version 20231120)
+	(version 20250114)
 	(generator "eeschema")
-	(generator_version "8.0")
+	(generator_version "9.0")
 	(paper "USLetter")
 	(title_block
 		(title "HMS Multichannel Olfactometer Driver")
-		(date "2025-01-23")
+		(date "2025-08-27")
 		(rev "4.1")
 		(company "HMS Research Instrumentation Core")
@@
 		(dnp no)
 		(fields_autoplaced yes)
-		(property "Reference" "U2"
+		(property "Reference" "U12"
 			(at 91.44 25.4 0)
 			(effects
@@
 		(dnp no)
 		(fields_autoplaced yes)
-		(property "Reference" "H7"
+		(property "Reference" "H12"
 			(at 55.88 100.3299 0)
 			(effects
@@
 		(dnp no)
 		(fields_autoplaced yes)
-		(property "Reference" "#PWR02"
+		(property "Reference" "#PWR029"
 			(at 91.44 67.31 0)
 			(effects
@@
 		(dnp no)
 		(fields_autoplaced yes)
-		(property "Reference" "#PWR05"
+		(property "Reference" "#PWR028"
 			(at 129.54 34.29 0)
 			(effects
@@
 		(dnp no)
 		(fields_autoplaced yes)
-		(property "Reference" "H1"
+		(property "Reference" "H6"
 			(at 55.88 95.2499 0)
 			(effects
@@
 		(dnp no)
 		(fields_autoplaced yes)
-		(property "Reference" "#PWR0101"
+		(property "Reference" "#PWR026"
 			(at 48.26 31.75 0)
 			(effects
@@
 		(dnp no)
 		(fields_autoplaced yes)
-		(property "Reference" "U3"
+		(property "Reference" "U13"
 			(at 50.4541 27.94 0)
 			(effects
@@
 		(dnp no)
 		(fields_autoplaced yes)
-		(property "Reference" "#PWR0102"
+		(property "Reference" "#PWR030"
 			(at 48.26 69.85 0)
 			(effects
@@
 		(dnp no)
 		(fields_autoplaced yes)
-		(property "Reference" "#PWR04"
+		(property "Reference" "#PWR027"
 			(at 104.14 34.29 0)
 			(effects
@@
 		(dnp no)
 		(fields_autoplaced yes)
-		(property "Reference" "J1"
+		(property "Reference" "J6"
 			(at 139.7 63.4999 0)
 			(effects
